File: HW2/Homework2/hw2.sch (EAGLE design)
At the start: 3 parts, among them J1 USBSMD

Commit message: schematic
Parts:
- added C1, C3, C4, C5: 0.1uF, Yuling:C-US025-024X044
- added C2, C6: 10uF, Yuling:C-US025-024X044
- added J2: RESET, Yuling:M02-JST-2-PTH-NO_SILK
- added J3, J4: (no value), Yuling:M08
- added J5: (no value), Yuling:M05PTH
- added LED1: Red, Yuling:LED3MM
- added LED2: Green, Yuling:LED3MM
- added R1, R2: 330, Yuling:R-US_0204/5
- added R3, R4: 10k, Yuling:R-US_0204/5
- added U$3: SLIDE, Yuling:SLIDE
- added U$4: USB-PORT, Yuling:USB-PORT
- added U$5: RESONATOR, Yuling:RESONATOR
- J1: value USBSMD -> USER; device Yuling:USBSMD -> Yuling:M02-JST-2-PTH-NO_SILK
Connections:
- removed net N$3: U$1.3.A1
- removed net N$5: U$1.5.PGEC1/B1
- removed net N$6: U$1.6.B2
- removed net N$7: U$1.7.B3
- new net +3V3: C2.1, C3.1, C4.1, C5.1, J4.7, J5.2, LED1.A, U$1.13.VDD, U$1.23.VUSB3V3, U$1.28.AVDD, U$2.3.VOUT
- new net +5V: C1.1, J3.2, U$1.16.B7, U$2.2.VIN, U$3.3.OUT
- new net A0: J4.1, U$1.2.A0
- new net A1: J4.2, U$1.3.A1
- new net A4/LED: J4.6, LED2.A, U$1.12.A4
- new net B13: J3.6, U$1.24.B13
- new net B14: J3.7, U$1.25.B14
- new net B15: J3.8, U$1.26.B15
- new net B2: J4.3, U$1.6.B2
- new net B3: J4.4, U$1.7.B3
- new net B4/USER: J1.1, J4.5, R4.1, R4.2, U$1.11.B4
- new net B7: J3.3
- new net B8: J3.4, U$1.17.B8
- new net B9: J3.5, U$1.18.B9
- new net D+: U$1.21.D+/B10, U$4.P$5
- new net D-: U$1.22.D-/B11, U$4.P$4
- new net MCLR: J2.1, J5.1, R3.1, R3.2, U$1.1.MCLR
- new net N$11: LED1.C, R1.2
- new net N$12: LED2.C, R2.2
- new net N$8: U$3.2.IN, U$4.P$3
- new net PGC: J5.5, U$1.5.PGEC1/B1
- new net PGD: J5.4, U$1.4.PGED1/B0
- new net USBID: U$1.14.USBID/B5, U$4.P$1
- net GND: now also C1.2, C2.2, C3.2, C4.2, C5.2, C6.2, J1.2, J2.2, J3.1, J4.8, J5.3, R1.1, R2.1, U$1.19.VSS, U$1.27.AVSS, U$2.1.GND, U$4.P$2, U$5.2.GND
- net N$1: now also U$5.1.OSC1; no longer U$1.1.MCLR
- net N$2: now also U$5.3.OSC2; no longer U$1.2.A0
- net N$4: now also C6.1, U$1.20.VCAP; no longer U$1.4.PGED1/B0
Other:
- moved on the sheet: U$2

Commit message: board
Connections:
- net +3V3: now also R3.2
- net MCLR: no longer R3.2
- net N$1: now also U$1.9.A2
- net N$2: now also U$1.10.A3
Changed lines of the file:
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@@
 <instance part="GND7" gate="1" x="187.96" y="76.2"/>
 <instance part="GND8" gate="1" x="187.96" y="43.18"/>
-<instance part="GND10" gate="1" x="43.18" y="20.32"/>
+<instance part="GND10" gate="1" x="53.34" y="20.32"/>
 <instance part="GND11" gate="1" x="48.26" y="68.58"/>
 <instance part="GND13" gate="1" x="53.34" y="-25.4"/>
@@
 <pinref part="C5" gate="G$1" pin="2"/>
 <pinref part="GND10" gate="1" pin="GND"/>
-<wire x1="53.34" y1="22.86" x2="43.18" y2="22.86" width="0.1524" layer="91"/>
 <pinref part="U$1" gate="G$1" pin="27.AVSS"/>
-<wire x1="43.18" y1="22.86" x2="30.48" y2="22.86" width="0.1524" layer="91"/>
-<junction x="43.18" y="22.86"/>
+<wire x1="53.34" y1="22.86" x2="30.48" y2="22.86" width="0.1524" layer="91"/>
+<junction x="53.34" y="22.86"/>
 </segment>
 <segment>
@@
 <net name="MCLR" class="0">
 <segment>
-<pinref part="+3V3" gate="G$1" pin="+3V3"/>
 <pinref part="J2" gate="G$1" pin="1"/>
-<wire x1="187.96" y1="68.58" x2="187.96" y2="58.42" width="0.1524" layer="91"/>
 <wire x1="187.96" y1="58.42" x2="187.96" y2="55.88" width="0.1524" layer="91"/>
 <wire x1="187.96" y1="55.88" x2="172.72" y2="55.88" width="0.1524" layer="91"/>
 <junction x="187.96" y="55.88"/>
 <label x="172.72" y="55.88" size="1.778" layer="95"/>
-<pinref part="R3" gate="G$1" pin="2"/>
-<junction x="187.96" y="68.58"/>
 <pinref part="R3" gate="G$1" pin="1"/>
-<junction x="187.96" y="58.42"/>
 </segment>
 <segment>
@@
 <wire x1="132.08" y1="12.7" x2="149.86" y2="12.7" width="0.1524" layer="91"/>
 </segment>
-</net>
-<net name="N$1" class="0">
-<segment>
-<pinref part="U$5" gate="G$1" pin="1.OSC1"/>
-<wire x1="-33.02" y1="-12.7" x2="-2.54" y2="-12.7" width="0.1524" layer="91"/>
-</segment>
-</net>
-<net name="N$2" class="0">
-<segment>
-<pinref part="U$5" gate="G$1" pin="3.OSC2"/>
-<wire x1="-33.02" y1="-22.86" x2="-20.32" y2="-22.86" width="0.1524" layer="91"/>
-<wire x1="-20.32" y1="-22.86" x2="-20.32" y2="-17.78" width="0.1524" layer="91"/>
-<wire x1="-20.32" y1="-17.78" x2="-2.54" y2="-17.78" width="0.1524" layer="91"/>
+<segment>
+<pinref part="+3V3" gate="G$1" pin="+3V3"/>
+<pinref part="R3" gate="G$1" pin="2"/>
 </segment>
 </net>
@@
 </segment>
 </net>
+<net name="N$1" class="0">
+<segment>
+<pinref part="U$5" gate="G$1" pin="1.OSC1"/>
+<wire x1="-33.02" y1="-12.7" x2="-5.08" y2="-12.7" width="0.1524" layer="91"/>
+<pinref part="U$1" gate="G$1" pin="9.A2"/>
+<wire x1="-5.08" y1="-12.7" x2="-2.54" y2="-12.7" width="0.1524" layer="91"/>
+<junction x="-5.08" y="-12.7"/>
+</segment>
+</net>
+<net name="N$2" class="0">
+<segment>
+<pinref part="U$5" gate="G$1" pin="3.OSC2"/>
+<wire x1="-33.02" y1="-22.86" x2="-17.78" y2="-22.86" width="0.1524" layer="91"/>
+<wire x1="-17.78" y1="-22.86" x2="-17.78" y2="-17.78" width="0.1524" layer="91"/>
+<wire x1="-17.78" y1="-17.78" x2="-5.08" y2="-17.78" width="0.1524" layer="91"/>
+<pinref part="U$1" gate="G$1" pin="10.A3"/>
+<wire x1="-5.08" y1="-17.78" x2="-2.54" y2="-17.78" width="0.1524" layer="91"/>
+<junction x="-5.08" y="-17.78"/>
+</segment>
+</net>
