File: HW2/Homework2/hw2.brd (EAGLE design)
At the start: 50 x 50 mm, 22 parts, among them J1 USER, J2 RESET

Commit message: Ready to be checked before order #I don’t really trust my design though. May I just use yours?
Routing:
- net D+: track 39.2 -> 39.9 mm, vias 1 -> 2
- net PGD: vias 2 -> 3
Changed lines of the file:
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@@
 </class>
 </classes>
-<designrules name="default">
+<designrules name="SeeedStudio_2layer_DRU_no_angle_20140221">
 <description language="de">&lt;b&gt;EAGLE Design Rules&lt;/b&gt;
 &lt;p&gt;
@@
 necessary adjustments and save your customized
 design rules under a new name.</description>
+<description language="zh">&lt;b&gt;Seeed Studio EAGLE Design Rules&lt;/b&gt;
+</description>
 <param name="layerSetup" value="(1*16)"/>
-<param name="mtCopper" value="0.035mm 0.035mm 0.035mm 0.035mm 0.035mm 0.035mm 0.035mm 0.035mm 0.035mm 0.035mm 0.035mm 0.035mm 0.035mm 0.035mm 0.035mm 0.035mm"/>
-<param name="mtIsolate" value="1.5mm 0.15mm 0.2mm 0.15mm 0.2mm 0.15mm 0.2mm 0.15mm 0.2mm 0.15mm 0.2mm 0.15mm 0.2mm 0.15mm 0.2mm"/>
-<param name="mdWireWire" value="8mil"/>
-<param name="mdWirePad" value="8mil"/>
-<param name="mdWireVia" value="8mil"/>
-<param name="mdPadPad" value="8mil"/>
-<param name="mdPadVia" value="8mil"/>
-<param name="mdViaVia" value="8mil"/>
-<param name="mdSmdPad" value="8mil"/>
-<param name="mdSmdVia" value="8mil"/>
-<param name="mdSmdSmd" value="8mil"/>
+<param name="mtCopper" value="0.035mm 0.0175mm 0.035mm 0.035mm 0.035mm 0.035mm 0.035mm 0.035mm 0.035mm 0.035mm 0.035mm 0.035mm 0.035mm 0.035mm 0.0175mm 0.035mm"/>
+<param name="mtIsolate" value="1.5mm 1.1mm 0.2mm 0.15mm 0.2mm 0.15mm 0.2mm 0.15mm 0.2mm 0.15mm 0.2mm 0.15mm 0.2mm 0.15mm 0.2mm"/>
+<param name="mdWireWire" value="6mil"/>
+<param name="mdWirePad" value="6mil"/>
+<param name="mdWireVia" value="6mil"/>
+<param name="mdPadPad" value="6mil"/>
+<param name="mdPadVia" value="6mil"/>
+<param name="mdViaVia" value="6mil"/>
+<param name="mdSmdPad" value="0mil"/>
+<param name="mdSmdVia" value="0mil"/>
+<param name="mdSmdSmd" value="0mil"/>
 <param name="mdViaViaSameLayer" value="8mil"/>
 <param name="mnLayersViaInSmd" value="2"/>
-<param name="mdCopperDimension" value="40mil"/>
-<param name="mdDrill" value="8mil"/>
+<param name="mdCopperDimension" value="10mil"/>
+<param name="mdDrill" value="10mil"/>
 <param name="mdSmdStop" value="0mil"/>
-<param name="msWidth" value="10mil"/>
-<param name="msDrill" value="24mil"/>
-<param name="msMicroVia" value="9.99mm"/>
+<param name="msWidth" value="6mil"/>
+<param name="msDrill" value="12mil"/>
+<param name="msMicroVia" value="12mil"/>
 <param name="msBlindViaRatio" value="0.5"/>
 <param name="rvPadTop" value="0.25"/>
@@
 <param name="rlMinPadBottom" value="10mil"/>
 <param name="rlMaxPadBottom" value="20mil"/>
-<param name="rlMinViaOuter" value="8mil"/>
+<param name="rlMinViaOuter" value="6mil"/>
 <param name="rlMaxViaOuter" value="20mil"/>
-<param name="rlMinViaInner" value="8mil"/>
+<param name="rlMinViaInner" value="6mil"/>
 <param name="rlMaxViaInner" value="20mil"/>
 <param name="rlMinMicroViaOuter" value="4mil"/>
@@
 <param name="psTop" value="-1"/>
 <param name="psBottom" value="-1"/>
-<param name="psFirst" value="-1"/>
+<param name="psFirst" value="0"/>
 <param name="psElongationLong" value="100"/>
 <param name="psElongationOffset" value="100"/>
 <param name="mvStopFrame" value="1"/>
 <param name="mvCreamFrame" value="0"/>
-<param name="mlMinStopFrame" value="4mil"/>
-<param name="mlMaxStopFrame" value="4mil"/>
+<param name="mlMinStopFrame" value="2mil"/>
+<param name="mlMaxStopFrame" value="2mil"/>
 <param name="mlMinCreamFrame" value="0mil"/>
 <param name="mlMaxCreamFrame" value="0mil"/>
-<param name="mlViaStopLimit" value="0mil"/>
+<param name="mlViaStopLimit" value="100mil"/>
 <param name="srRoundness" value="0"/>
 <param name="srMinRoundness" value="0mil"/>
@@
 <param name="checkAngle" value="0"/>
 <param name="checkFont" value="1"/>
-<param name="checkRestrict" value="1"/>
+<param name="checkRestrict" value="0"/>
 <param name="useDiameter" value="13"/>
 <param name="maxErrors" value="50"/>
@@
 <wire x1="21.59" y1="31.75" x2="22.86" y2="31.75" width="0.4064" layer="1"/>
 <wire x1="22.86" y1="31.75" x2="24.13" y2="33.02" width="0.4064" layer="1"/>
-<wire x1="24.13" y1="33.02" x2="35.56" y2="33.02" width="0.4064" layer="1"/>
 <via x="35.56" y="33.02" extent="1-16" drill="0.5" shape="octagon"/>
-<wire x1="35.56" y1="33.02" x2="46.99" y2="33.02" width="0.4064" layer="16"/>
 <via x="46.99" y="33.02" extent="1-16" drill="0.5" shape="octagon"/>
 <wire x1="46.99" y1="33.02" x2="46.99" y2="44.45" width="0.4064" layer="1"/>
 <wire x1="46.99" y1="44.45" x2="48.895" y2="44.45" width="0.4064" layer="1"/>
+<wire x1="24.13" y1="33.02" x2="26.035" y2="33.02" width="0.4064" layer="1"/>
+<via x="26.035" y="33.02" extent="1-16" drill="0.5" shape="octagon"/>
+<wire x1="26.035" y1="33.02" x2="46.99" y2="33.02" width="0.4064" layer="16"/>
+<wire x1="26.035" y1="33.02" x2="35.56" y2="33.02" width="0" layer="19" extent="16-16"/>
 </signal>
 <signal name="PGC">
@@
 <wire x1="11.7475" y1="45.4025" x2="12.7" y2="44.45" width="0.4064" layer="1"/>
 <wire x1="12.7" y1="44.45" x2="12.7" y2="34.29" width="0.4064" layer="1"/>
-<wire x1="12.7" y1="34.29" x2="19.05" y2="27.94" width="0.4064" layer="1"/>
-<wire x1="19.05" y1="27.94" x2="24.13" y2="27.94" width="0.4064" layer="1"/>
-<wire x1="24.13" y1="27.94" x2="24.13" y2="21.59" width="0.4064" layer="1"/>
 <via x="24.13" y="21.59" extent="1-16" drill="0.5" shape="octagon"/>
 <wire x1="24.13" y1="21.59" x2="29.21" y2="21.59" width="0.4064" layer="16"/>
+<wire x1="24.13" y1="21.59" x2="24.13" y2="27.94" width="0.4064" layer="16"/>
+<wire x1="24.13" y1="27.94" x2="17.78" y2="27.94" width="0.4064" layer="16"/>
+<via x="17.78" y="27.94" extent="1-16" drill="0.5" shape="octagon"/>
+<wire x1="17.78" y1="27.94" x2="17.78" y2="29.21" width="0.4064" layer="1"/>
+<wire x1="17.78" y1="29.21" x2="12.7" y2="34.29" width="0.4064" layer="1"/>
 </signal>
 <signal name="B9">
@@
 </signal>
 </signals>
+<errors>
+</errors>
 </board>
 </drawing>
